File: head_amp.kicad_pcb (KiCad board)
At the start: 2 copper layers, 63 parts, among them J1 USB Interface, J3 AudioJack4, M1 Fan, Q1 AO3401A, Q2 BSS138, Q3 LRC L8050QLT1G, Q4 LRC L8050QLT1G, U1 TXS0102DCU, U2 CH340K, U3 Digital Regulator, U4 Analog Regulator, U5 TXS0102DCU, U6 ESP32-S3-WROOM-1, U7 LSM6DS3, U8 WM8988LGECN/V, U9 WM8988LGECN/V

Commit message: More stuff
Parts:
- removed Q3, Q4: LRC L8050QLT1G, Package_TO_SOT_SMD:SOT-23
- removed TP1: Boot, TestPoint:TestPoint_2Pads_Pitch5.08mm_Drill1.3mm
- removed TP2: Reset, TestPoint:TestPoint_2Pads_Pitch5.08mm_Drill1.3mm
- removed U9: WM8988LGECN/V, footprints:QFN28_4X4_CIR-M
- added C34: 4.7u, Capacitor_SMD:C_0603_1608Metric, F.Cu at (96.8, 89.0)
- added C35: 4.7u, Capacitor_SMD:C_0603_1608Metric, F.Cu at (96.8, 91.5)
- added C36: 1u, Capacitor_SMD:C_0603_1608Metric, F.Cu at (96.8, 94.0)
- added J2: Left_Mic, Connector_JST:JST_XH_S2B-XH-A_1x02_P2.50mm_Horizontal, F.Cu at (139.0, 22.2)
- added J4: AudioJack4, Connector_Audio:Jack_3.5mm_PJ320D_Horizontal, F.Cu at (144.8, 55.5)
- added R11: 10k, Resistor_SMD:R_0603_1608Metric, F.Cu at (149.6, 43.7)
- added SW1: Boot, Button_Switch_THT:SW_Tactile_SPST_Angled_PTS645Vx39-2LFS, F.Cu at (134.8, 119.5)
- added SW2: Reset, Button_Switch_THT:SW_Tactile_SPST_Angled_PTS645Vx39-2LFS, F.Cu at (165.8, 119.5)
- C11: value 1u -> 2.2u
- C12, C16, C6: value 1u -> 100n
- C13, C27, C9: value 100n -> 1u
- C14: value 2.2u -> 100n
- C17, C18: value 100n -> 220u; footprint Capacitor_SMD:C_0603_1608Metric -> Capacitor_SMD:CP_Elec_5x5.4
- C21: value 100n -> 4.7u; footprint Capacitor_SMD:C_0603_1608Metric -> Capacitor_SMD:CP_Elec_5x4.5
- C23, C30, C31: footprint Capacitor_SMD:C_0603_1608Metric -> Capacitor_SMD:CP_Elec_5x4.5
- C24: value 4.7u -> 1u
- C25, C26: footprint Capacitor_SMD:CP_Elec_5x4.5 -> Capacitor_SMD:C_0603_1608Metric
- C29: value 4.7u -> 100n; footprint Capacitor_SMD:CP_Elec_5x4.5 -> Capacitor_SMD:C_0603_1608Metric
- C33: value 4.7u -> 1u; footprint Capacitor_SMD:CP_Elec_5x4.5 -> Capacitor_SMD:C_0603_1608Metric
- C5: value 100n -> 2.2u
- C8: value 2.2u -> 1u
- J3: value AudioJack4 -> Right_Mic; footprint Connector_Audio:Jack_3.5mm_PJ320D_Horizontal -> Connector_JST:JST_XH_S2B-XH-A_1x02_P2.50mm_Horizontal
- Q1: value AO3401A -> LRC L8050QLT1G
- Q2: value BSS138 -> LRC L8050QLT1G
- R10: value 1k -> 10k
- R2: value 5.1k -> 10k
- R3, R4: value 10k -> 22
- R5, R6: value 22 -> 5.1k
- R7, R8: value 5.1k -> 1k
- R9: value 1k -> 0; footprint Resistor_SMD:R_0603_1608Metric -> Resistor_SMD:R_2512_6332Metric
- U1: value TXS0102DCU -> CH340K; footprint Package_SO:VSSOP-8_2.3x2mm_P0.5mm -> Package_SO:SSOP-10-1EP_3.9x4.9mm_P1mm_EP2.1x3.3mm
- U2: value CH340K -> Digital Regulator; footprint Package_SO:SSOP-10-1EP_3.9x4.9mm_P1mm_EP2.1x3.3mm -> Package_TO_SOT_SMD:TO-252-2
- U3: value Digital Regulator -> Analog Regulator
- U4: value Analog Regulator -> TXS0102DCU; footprint Package_TO_SOT_SMD:TO-252-2 -> Package_SO:VSSOP-8_2.3x2mm_P0.5mm
- U5: value TXS0102DCU -> ESP32-S3-WROOM-1; footprint Package_SO:VSSOP-8_2.3x2mm_P0.5mm -> RF_Module:ESP32-S3-WROOM-1
- U6: value ESP32-S3-WROOM-1 -> LSM6DS3; footprint RF_Module:ESP32-S3-WROOM-1 -> Package_LGA:LGA-14_3x2.5mm_P0.5mm_LayoutBorder3x4y
- U7: value LSM6DS3 -> WM8988LGECN/V; footprint Package_LGA:LGA-14_3x2.5mm_P0.5mm_LayoutBorder3x4y -> footprints:QFN28_4X4_CIR-M
- moved C21 126.3 mm to (73.1, 77.4)
- moved C23 125.1 mm to (73.1, 91.1)
- moved C8 121.6 mm to (141.5, 33.7)
- moved J3 121.5 mm to (148.4, 22.2)
- moved C27 120.5 mm to (79.6, 94.0)
- moved C24 119.3 mm to (79.6, 86.5)
- moved C15 119.1 mm to (145.6, 33.7)
- moved C16 119.1 mm to (145.6, 36.2)
- moved C22 119.0 mm to (73.1, 84.2)
- moved C20 118.8 mm to (79.6, 84.0)
- moved C30 116.5 mm to (90.3, 77.4)
- moved C31 114.9 mm to (90.3, 84.2)
- moved C26 113.4 mm to (79.6, 91.5)
- moved C25 112.8 mm to (79.6, 89.0)
- moved U7 109.8 mm to (82.4, 74.9)
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Connections:
- C11 pad 1: VBUS -> +3V3A
- C11 pad 2: GND -> GNDA
- C12 pad 2: +3V3D -> VBUS
- C13 pad 2: +3V3D -> VBUS
- C14 pad 1: +3V3A -> VBUS
- C15 pad 1: GND -> +3V3D
- C15 pad 2: VBUS -> GND
- C16 pad 1: GND -> +3V3D
- C16 pad 2: VBUS -> GND
- C17 pad 1: VBUS -> /Ext->Int/OUT_Right
- C17 pad 2: GND -> /Headset_Right
- C18 pad 1: +3V3D -> /Ext->Int/OUT_Left
- C18 pad 2: GND -> /Headset_Left
- C19 pad 1: +3V3D -> GND
- C19 pad 2: GND -> +3V3D
- C2 pad 1: GND -> Net-(U1-V3)
- C2 pad 2: VBUS -> GND
- C21 pad 1: GND -> Net-(U7-HPCOM)
- C21 pad 2: +3V3D -> GNDA
- C22 pad 1: Net-(U8-HPCOM) -> Net-(U7-VMID)
- C23 pad 1: GND -> Net-(U7-VREF)
- C23 pad 2: Net-(U8-VMID) -> GND
- C24 pad 1: GND -> /Mic_Left
- C24 pad 2: Net-(U8-VREF) -> Net-(U7-LINPUT1)
- C25 pad 1: +3V3A -> GNDA
- C25 pad 2: GND -> +3V3A
- C26 pad 1: +3V3A -> GNDA
- C26 pad 2: GND -> +3V3A
- C27 pad 1: GND -> /Mic_Right
- C27 pad 2: +3V3D -> Net-(U7-RINPUT1)
- C29 pad 1: Net-(U9-HPCOM) -> GND
- C29 pad 2: GND -> +3V3D
- C3 pad 1: GND -> VBUS
- C3 pad 2: VBUS -> GND
- C30 pad 1: GND -> Net-(U8-HPCOM)
- C30 pad 2: Net-(U9-VMID) -> GNDA
- C31 pad 1: GND -> Net-(U8-VMID)
- C31 pad 2: Net-(U9-VREF) -> GND
- C32 pad 1: +3V3A -> Net-(U8-VREF)
- C33 pad 1: +3V3A -> /Headset_Mic
- C33 pad 2: GND -> Net-(U8-LINPUT1)
- C4 pad 1: GND -> /GPIO0
- C4 pad 2: +3V3D -> GND
- C5 pad 1: Net-(U2-V3) -> +3V3D
- C6 pad 1: VBUS -> /MCU_EN
- C7 pad 1: /GPIO0 -> GND
- C7 pad 2: GND -> +3V3D
- C8 pad 1: +3V3D -> VBUS
- C8 pad 2: GND -> GNDA
- C9 pad 1: /MCU_EN -> GND
- C9 pad 2: GND -> +3V3D
- Q1 pad 1: /FAN_PWM -> Net-(Q1-B)
- Q1 pad 2: VBUS -> /RTS
- Q1 pad 3: Net-(Q1-D) -> /MCU_EN
- Q2 pad 1: /FAN_PWM -> Net-(Q2-B)
- Q2 pad 2: GND -> /DTR
- Q2 pad 3: Net-(Q1-D) -> /GPIO0
- R1 pad 1: /FAN_RPM -> /DTR
- R1 pad 2: GND -> Net-(Q1-B)
- R10 pad 1: /MCU_TX -> /Mic_Left
- R10 pad 2: Net-(D2-K) -> VDD
- R2 pad 1: unconnected-(R2-Pad1) -> /RTS
- R2 pad 2: /FAN_RPM -> Net-(Q2-B)
- R3 pad 1: /DTR -> Net-(J1-D--PadA7)
- R3 pad 2: Net-(Q3-B) -> /USB_D-
- R4 pad 1: /RTS -> Net-(J1-D+-PadA6)
- R4 pad 2: Net-(Q4-B) -> /USB_D+
- R5 pad 1: Net-(J1-D--PadA7) -> Net-(J1-CC1)
- R5 pad 2: /USB_D- -> GND
- R6 pad 1: Net-(J1-D+-PadA6) -> Net-(J1-CC2)
- R6 pad 2: /USB_D+ -> GND
- R7 pad 1: Net-(J1-CC1) -> /MCU_RX
- R7 pad 2: GND -> Net-(D1-K)
- R8 pad 1: Net-(J1-CC2) -> /MCU_TX
- R8 pad 2: GND -> Net-(D2-K)
- R9 pad 1: /MCU_RX -> GND
- R9 pad 2: Net-(D1-K) -> GNDA
- U1 pad 1: unconnected-(U1-B2-Pad1) -> /USB_D+
- U1 pad 2: GND -> /USB_D-
- U1 pad 3: +3V3D -> GND
- U1 pad 4: /FAN_PWM -> /DTR
- U1 pad 5: /FAN_RPM -> unconnected-(U1-~{CTS}-Pad5)
- U1 pad 6: +3V3D -> /RTS
- U1 pad 7: VBUS -> +3V3D
- U1 pad 8: unconnected-(U1-B1-Pad8) -> /MCU_RX
- U2 pad 1: /USB_D+ -> GND
- U2 pad 2: /USB_D- -> +3V3D
- U2 pad 3: GND -> VBUS
- U3 pad 1: GND -> GNDA
- U3 pad 2: +3V3D -> +3V3A
- U4 pad 1: GND -> Net-(M1-PWM)
- U4 pad 2: +3V3A -> GND
- U4 pad 3: VBUS -> +3V3D
- U5 pad 1: Net-(M1-PWM) -> GND
- U5 pad 2: GND -> +3V3D
- U5 pad 3: +3V3D -> /MCU_EN
- U5 pad 4: /FAN_PWM -> unconnected-(U5-IO4-Pad4)
- U5 pad 5: /FAN_RPM -> unconnected-(U5-IO5-Pad5)
- U5 pad 6: +3V3D -> unconnected-(U5-IO6-Pad6)
- U5 pad 7: VBUS -> unconnected-(U5-IO7-Pad7)
- U5 pad 8: Net-(M1-Tacho) -> unconnected-(U5-IO15-Pad8)
- U6 pad 1: GND -> /MISO
- U6 pad 12: unconnected-(U6-IO8-Pad12) -> /IMU_Select
- U6 pad 13: unconnected-(U6-USB_D--Pad13) -> /SPI_CLK
- U6 pad 14: unconnected-(U6-USB_D+-Pad14) -> /MOSI
- U6 pad 2: +3V3D -> GND
- U6 pad 3: /MCU_EN -> GND
- U6 pad 5: unconnected-(U6-IO5-Pad5) -> +3V3D
- U6 pad 6: unconnected-(U6-IO6-Pad6) -> GND
- U6 pad 7: unconnected-(U6-IO7-Pad7) -> GND
- U6 pad 8: unconnected-(U6-IO15-Pad8) -> +3V3D
- U7 pad 1: /MISO -> /Ext->Int/Master_CLK
- U7 pad 11: unconnected-(U7-NC-Pad11) -> /Ext->Int/OUT_Right
- U7 pad 12: /IMU_Select -> /Ext->Int/OUT_Left
- U7 pad 13: /SPI_CLK -> GNDA
- U7 pad 14: /MOSI -> unconnected-(U7-ROUT2-Pad14)
- U7 pad 2: unconnected-(U7-SDX-Pad2) -> +3V3D
- U7 pad 3: unconnected-(U7-SCX-Pad3) -> +3V3D
- U7 pad 4: unconnected-(U7-INT1-Pad4) -> GND
- U7 pad 5: +3V3D -> /Ext->Int_CLK
- U7 pad 6: GND -> /Ext->Int_In
- U7 pad 7: GND -> /Ext->Int_LRC
- U7 pad 8: +3V3D -> /Ext->Int_Out
- U7 pad 9: unconnected-(U7-INT2-Pad9) -> Net-(U7-HPCOM)
- U8 pad 1: /Ext->Int/Master_CLK -> /Int->Ext/Master_CLK
- U8 pad 11: /Headset_Right -> /Int->Ext/OUT_Right
- U8 pad 12: /Headset_Left -> /Int->Ext/OUT_Left
- U8 pad 13: GND -> GNDA
- U8 pad 18: GND -> GNDA
- U8 pad 23: /Ext->Int/IN_Right -> Net-(U8-RINPUT1)
- U8 pad 24: /Ext->Int/IN_Left -> Net-(U8-LINPUT1)
- U8 pad 26: /Exit->Int_Select -> /Int->Ext_Select
- U8 pad 5: /Ext->Int_CLK -> /Int->Ext_CLK
- U8 pad 6: /Ext->Int_In -> /Int->Ext_In
- U8 pad 7: /Ext->Int_LRC -> /Int->Ext_LRC
- U8 pad 8: /Ext->Int_Out -> /Int->Ext_Out
Routing:
- net /MCU_EN: track 0.00 -> 57.1 mm, vias 0 -> 1
- net /MCU_TX: track 0.00 -> 43.6 mm, vias 0 -> 2
- net GND: track 0.00 -> 41.1 mm, vias 0 -> 5
- net /GPIO0: track 0.00 -> 36.0 mm
- net /MCU_RX: track 0.00 -> 28.8 mm, vias 0 -> 2
- net /RTS: track 0.00 -> 7.99 mm
- net /DTR: track 0.00 -> 6.80 mm
- net VBUS: track 0.00 -> 4.40 mm
- net Net-(U1-V3): track 0.00 -> 4.19 mm
- net +3V3D: track 0.00 -> 3.78 mm
- net /USB_D-: track 0.00 -> 3.13 mm
- net /USB_D+: track 0.00 -> 2.71 mm
- net Net-(Q2-B): track 0.00 -> 2.39 mm
- net Net-(Q1-B): track 0.00 -> 2.00 mm
- net Net-(D2-K): track 0.00 -> 1.35 mm
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- added copper zone on B.Cu, net GND
Other:
- board outline added: 215 x 161 mm

Commit message: Fixes
Parts:
- removed the C17 at (137.5, 64.5)
- removed the C35 at (96.8, 91.5)
- added C20: 4.7u, Capacitor_SMD:CP_Elec_5x4.5, F.Cu at (52.9, 77.5)
- added C33: 4.7u, Capacitor_SMD:CP_Elec_5x4.5, F.Cu at (63.8, 91.2)
- added C37: 4.7u, Capacitor_SMD:C_0603_1608Metric, F.Cu at (70.3, 73.5)
- added C38: 1u, Capacitor_SMD:C_0603_1608Metric, F.Cu at (70.3, 76.0)
- added J2: Left_Speaker, Connector_JST:JST_XH_S2B-XH-A_1x02_P2.50mm_Horizontal, F.Cu at (164.8, 22.0)
- added J6: AudioJack4, Connector_Audio:Jack_3.5mm_PJ320D_Horizontal, F.Cu at (162.1, 61.8)
- added R12: 10k, Resistor_SMD:R_0603_1608Metric, F.Cu at (163.4, 33.5)
- C21, C32: value 4.7u -> 220u; footprint Capacitor_SMD:CP_Elec_5x4.5 -> Capacitor_SMD:CP_Elec_5x5.4
- C29: value 100n -> 220u; footprint Capacitor_SMD:C_0603_1608Metric -> Capacitor_SMD:CP_Elec_5x5.4
- C30: value 4.7u -> 100n; footprint Capacitor_SMD:CP_Elec_5x4.5 -> Capacitor_SMD:C_0603_1608Metric
- C34: footprint Capacitor_SMD:C_0603_1608Metric -> Capacitor_SMD:CP_Elec_5x4.5
- C36: value 1u -> 4.7u
- J4: value AudioJack4 -> Right_Speaker; footprint Connector_Audio:Jack_3.5mm_PJ320D_Horizontal -> Connector_JST:JST_XH_S2B-XH-A_1x02_P2.50mm_Horizontal
- moved C18 84.7 mm to (52.9, 70.6)
- moved U3 77.1 mm to (170.4, 76.4)
- moved C3 73.4 mm to (168.9, 105.0), turned to 180 degrees
- moved C5 63.1 mm to (164.8, 100.6), turned to -90 degrees
- moved U2 58.4 mm to (169.5, 97.6)
- moved U7 55.2 mm to (135.2, 91.0), turned to 90 degrees
- moved C35 52.3 mm to (146.0, 68.8), turned to -90 degrees
- moved J4 44.7 mm to (174.3, 22.0)
- moved U8 43.4 mm to (158.8, 90.9), turned to 90 degrees
- moved C29 35.6 mm to (63.8, 70.6)
- moved C36 35.1 mm to (70.3, 70.9)
- moved C34 34.2 mm to (63.8, 98.0)
- moved C31 27.3 mm to (63.8, 77.5)
- moved C32 27.3 mm to (63.8, 84.3)
- moved U4 23.6 mm to (148.4, 97.8)
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- renumbered C19 to C17, C20 to C19, C33 to C35, J2 to J3, J3 to J5
Connections:
- C18 pad 1: /Ext->Int/OUT_Left -> Net-(U7-ROUT1)
- C18 pad 2: /Headset_Left -> /Headset_Right
- C21 pad 1: Net-(U7-HPCOM) -> Net-(U7-LOUT1)
- C21 pad 2: GNDA -> /Headset_Left
- C29 pad 1: GND -> Net-(U8-ROUT1)
- C29 pad 2: +3V3D -> /Speaker_Right
- C30 pad 1: Net-(U8-HPCOM) -> GND
- C30 pad 2: GNDA -> +3V3D
- C31 pad 1: Net-(U8-VMID) -> Net-(U8-HPCOM)
- C31 pad 2: GND -> GNDA
- C32 pad 1: Net-(U8-VREF) -> Net-(U8-LOUT1)
- C32 pad 2: GND -> /Speaker_Left
- C34 pad 1: GNDA -> Net-(U8-VREF)
- C34 pad 2: +3V3A -> GND
- C36 pad 1: /Headset_Mic -> GNDA
- C36 pad 2: Net-(U8-RINPUT1) -> +3V3A
- U7 pad 11: /Ext->Int/OUT_Right -> Net-(U7-ROUT1)
- U7 pad 12: /Ext->Int/OUT_Left -> Net-(U7-LOUT1)
- U8 pad 11: /Int->Ext/OUT_Right -> Net-(U8-ROUT1)
- U8 pad 12: /Int->Ext/OUT_Left -> Net-(U8-LOUT1)
Routing:
- net +3V3D: track 3.78 -> 23.6 mm, vias 0 -> 3
- net Net-(J1-CC1): track 0.00 -> 7.26 mm
- net Net-(J1-CC2): track 0.00 -> 7.05 mm
- net Net-(J1-D+-PadA6): track 0.00 -> 4.91 mm
- net Net-(J1-D--PadA7): track 0.00 -> 4.86 mm
- net /USB_D+: track 2.71 -> 6.63 mm
- net GND: track 41.1 -> 44.3 mm, vias 5 -> 7
- net /Headset_Mic: track 0.00 -> 2.11 mm
- net VBUS: track 4.40 -> 6.35 mm, vias 0 -> 3
- net GNDA: track 0.00 -> 0.96 mm, vias 0 -> 1
- added copper zone on In2.Cu, net +3V3A
- added copper zone on In2.Cu, net +3V3D
- added copper zone on B.Cu, net GNDA
- added copper zone on In1.Cu, net VBUS
Other:
- board size 215 x 161 mm -> 76 x 60 mm
- copper layers 2 -> 4

Commit message: started compact layout
Parts:
- removed D1: RX_LED, LED_SMD:LED_0603_1608Metric
- removed D2: TX_LED, LED_SMD:LED_0603_1608Metric
- removed R10, R11, R12: 10k, Resistor_SMD:R_0603_1608Metric
- C11, C5: value 2.2u -> 22u
- C20, C22, C23, C31, C33, C34: footprint Capacitor_SMD:CP_Elec_5x4.5 -> Capacitor_SMD:C_0603_1608Metric
- C3, C8: value 1u -> 10u
- R3, R4: value 22 -> 5.1k
- R5, R6: value 5.1k -> 22
- R7, R8: value 1k -> 10k
- R9: value 0 -> 10k; footprint Resistor_SMD:R_2512_6332Metric -> Resistor_SMD:R_0603_1608Metric
- moved C33 118.0 mm to (181.4, 100.8)
- moved C31 116.3 mm to (178.0, 99.3), turned to 90 degrees
- moved C30 116.2 mm to (180.8, 104.3), turned to 180 degrees
- moved C34 111.7 mm to (175.5, 95.8), turned to 90 degrees
- moved C36 111.7 mm to (179.0, 96.7)
- moved C37 111.2 mm to (177.5, 102.8), turned to 90 degrees
- moved C18 103.6 mm to (156.0, 80.2), turned to 90 degrees
- moved C29 94.1 mm to (156.0, 89.2), turned to 90 degrees
- moved C9 88.9 mm to (160.0, 123.2), turned to 180 degrees
- moved C10 88.0 mm to (160.0, 124.8), turned to 180 degrees
- moved C21 87.2 mm to (140.0, 80.2), turned to 90 degrees
- moved C20 83.3 mm to (133.5, 98.4), turned to 90 degrees
- moved C27 80.5 mm to (159.5, 84.8), turned to -90 degrees
- moved C38 78.0 mm to (146.3, 93.5)
- moved C15 77.3 mm to (115.2, 104.8)
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Connections:
- C22 pad 1: Net-(U7-VMID) -> GND
- C22 pad 2: GND -> Net-(U7-VMID)
- C23 pad 1: Net-(U7-VREF) -> GND
- C23 pad 2: GND -> Net-(U7-VREF)
- C33 pad 1: Net-(U8-VMID) -> GND
- C33 pad 2: GND -> Net-(U8-VMID)
- C34 pad 1: Net-(U8-VREF) -> GND
- C34 pad 2: GND -> Net-(U8-VREF)
- J1 pad A6: Net-(J1-D+-PadA6) -> /USB_D1+
- J1 pad A7: Net-(J1-D--PadA7) -> /USB_D1-
- J1 pad B6: Net-(J1-D+-PadA6) -> /USB_D1+
- J1 pad B7: Net-(J1-D--PadA7) -> /USB_D1-
- R3 pad 1: Net-(J1-D--PadA7) -> Net-(J1-CC1)
- R3 pad 2: /USB_D- -> GND
- R4 pad 1: Net-(J1-D+-PadA6) -> Net-(J1-CC2)
- R4 pad 2: /USB_D+ -> GND
- R5 pad 1: Net-(J1-CC1) -> /USB_D1-
- R5 pad 2: GND -> /USB_D-
- R6 pad 1: Net-(J1-CC2) -> /USB_D1+
- R6 pad 2: GND -> /USB_D+
- R7 pad 1: /MCU_RX -> /Mic_Left
- R7 pad 2: Net-(D1-K) -> +3V3A
- R8 pad 1: /MCU_TX -> /Mic_Right
- R8 pad 2: Net-(D2-K) -> +3V3A
- R9 pad 1: GND -> /Headset_Mic
- R9 pad 2: GNDA -> +3V3A
- U5 pad 4: unconnected-(U5-IO4-Pad4) -> /FAN_PWM
- U5 pad 5: unconnected-(U5-IO5-Pad5) -> /FAN_RPM
- U7 pad 25: +3V3 -> +3V3D
- U8 pad 25: +3V3 -> +3V3D
Routing:
- net Net-(U7-RINPUT1): track 0.00 -> 39.8 mm, vias 0 -> 2
- net /MCU_TX: track 43.6 -> 4.48 mm, vias 2 -> 0
- net /RTS: track 7.99 -> 42.9 mm
- net Net-(U7-ROUT1): track 0.00 -> 32.1 mm, vias 0 -> 2
- net /DTR: track 6.80 -> 35.7 mm
- net GND: track 44.3 -> 72.5 mm
- net /MCU_RX: track 28.8 -> 5.39 mm, vias 2 -> 0
- net +3V3A: track 0.00 -> 22.5 mm, vias 0 -> 4
- net /MCU_EN: track 57.1 -> 36.2 mm, vias 1 -> 2
- net VBUS: track 6.35 -> 26.0 mm, vias 3 -> 4
- net Net-(U7-LOUT1): track 0.00 -> 19.3 mm, vias 0 -> 2
- net Net-(U7-LINPUT1): track 0.00 -> 17.5 mm, vias 0 -> 2
- net GNDA: track 0.96 -> 17.6 mm, vias 1 -> 5
- net /Headset_Left: track 0.00 -> 16.4 mm
- net /USB_D1+: track 0.00 -> 9.79 mm
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Other:
- board size 76 x 60 mm -> 50 x 50 mm
