File: head_amp.kicad_pcb (KiCad board)
At the start: 4 copper layers, 50 x 50 mm, 49 parts, among them J1 Conn_01x15, J2 Conn_01x15, J3 Conn_01x03, J4 Conn_01x03, J5 Left_Speaker, J6 Left_Mic, J7 Right_Speaker, J8 Right_Mic, M1 Fan, Q1 AO3401A, Q2 AO3400A, U1 LSM6DS3, U2 Headphone Jack, U3 WM8988LGECN/V, U4 WM8988LGECN/V

Commit message: feat: pretty much done
Parts:
- removed C2, C3: 100n, Capacitor_SMD:C_0603_1608Metric
- removed U1: LSM6DS3, Package_LGA:LGA-14_3x2.5mm_P0.5mm_LayoutBorder3x4y
- added G***: LOGO, LOGO, B.Cu at (149.0, 114.5)
- added H1: MountingHole, MountingHole:MountingHole_2.2mm_M2, F.Cu at (141.0, 79.0)
- added H2: MountingHole, MountingHole:MountingHole_2.2mm_M2, F.Cu at (155.0, 79.0)
- added H3: MountingHole, MountingHole:MountingHole_2.2mm_M2, F.Cu at (156.0, 122.5)
- added H4: MountingHole, MountingHole:MountingHole_2.2mm_M2, F.Cu at (140.0, 122.5)
- added NT1: NetTie_2, NetTie:NetTie-2_THT_Pad1.0mm, F.Cu at (127.7, 117.0)
- added NT2: NetTie_2, NetTie:NetTie-2_THT_Pad1.0mm, F.Cu at (130.2, 120.0)
- J3: value Conn_01x03 -> Conn_01x05; footprint Connector_JST:JST_XH_S3B-XH-A_1x03_P2.50mm_Horizontal -> Connector_JST:JST_XH_S5B-XH-A_1x05_P2.50mm_Horizontal
- U3, U4: footprint footprints:QFN28_4X4_CIR-M -> footprints:QFN28_4X4_CIR
- moved C1 90.7 mm to (157.6, 112.0), turned to 90 degrees
- moved C4 86.0 mm to (152.8, 105.6), turned to 90 degrees
- moved C7 84.9 mm to (154.4, 105.6), turned to 90 degrees
- moved C8 80.8 mm to (157.0, 100.8), turned to 90 degrees
- moved C11 73.6 mm to (150.0, 99.8), turned to 90 degrees
- moved C12 70.7 mm to (148.5, 99.8), turned to 90 degrees
- moved C14 69.3 mm to (155.5, 96.2), turned to -90 degrees
- moved C15 66.4 mm to (153.9, 96.2), turned to -90 degrees
- moved U3 63.4 mm to (153.6, 100.8), turned to 90 degrees
- moved C20 59.0 mm to (144.2, 105.6), turned to 90 degrees
- moved C28 56.1 mm to (145.1, 96.3), turned to -90 degrees
- moved C27 54.5 mm to (143.5, 96.3), turned to -90 degrees
- moved C24 52.0 mm to (140.0, 99.8), turned to 90 degrees
- moved C21 47.1 mm to (147.0, 100.8)
- moved U4 43.6 mm to (143.4, 100.8)
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Connections:
- C10 pad 1: /Headset_Left -> /Speaker_Left
- C13 pad 1: /Mic_Left -> /Headset_Mic
- C16 pad 1: /Mic_Right -> /Headset_Mic
- C18 pad 1: /Speaker_Right -> /Headset_Right
- C19 pad 1: /Speaker_Right -> /Headset_Right
- C22 pad 1: /Speaker_Left -> /Headset_Left
- C23 pad 1: /Speaker_Left -> /Headset_Left
- C26 pad 1: /Headset_Mic -> /Mic_Left
- C29 pad 1: /Headset_Mic -> /Mic_Right
- C5 pad 1: /Headset_Right -> /Speaker_Right
- C6 pad 1: /Headset_Right -> /Speaker_Right
- C9 pad 1: /Headset_Left -> /Speaker_Left
- J1 pad 10: unconnected-(J1-Pin_10-Pad10) -> /MOSI
- J1 pad 11: unconnected-(J1-Pin_11-Pad11) -> /SPI_CLK
- J1 pad 12: unconnected-(J1-Pin_12-Pad12) -> /Master_Audio_Clk
- J1 pad 4: unconnected-(J1-Pin_4-Pad4) -> /LED_Data
- J1 pad 5: unconnected-(J1-Pin_5-Pad5) -> /Exit->Int_Select
- J1 pad 6: unconnected-(J1-Pin_6-Pad6) -> /Ext->Int_CLK
- J1 pad 7: unconnected-(J1-Pin_7-Pad7) -> /Ext->Int_In
- J1 pad 8: unconnected-(J1-Pin_8-Pad8) -> /Ext->Int_LRC
- J1 pad 9: unconnected-(J1-Pin_9-Pad9) -> /Ext->Int_Out
- J2 pad 3: unconnected-(J2-Pin_3-Pad3) -> /Out_DAT
- J2 pad 4: unconnected-(J2-Pin_4-Pad4) -> /Out_CLK
- J2 pad 5: unconnected-(J2-Pin_5-Pad5) -> /Int->Ext_Out
- J2 pad 6: unconnected-(J2-Pin_6-Pad6) -> /Int->Ext_LRC
- J2 pad 7: unconnected-(J2-Pin_7-Pad7) -> /Int->Ext_In
- J2 pad 8: unconnected-(J2-Pin_8-Pad8) -> /Int->Ext_CLK
- J2 pad 9: unconnected-(J2-Pin_9-Pad9) -> /Int->Ext_Select
- J3 pad 1: unconnected-(J3-Pin_1-Pad1) -> +5V
- J3 pad 2: unconnected-(J3-Pin_2-Pad2) -> +3V3D
- J3 pad 3: unconnected-(J3-Pin_3-Pad3) -> /Out_CLK
- J4 pad 1: unconnected-(J4-Pin_1-Pad1) -> +5V
- J4 pad 2: unconnected-(J4-Pin_2-Pad2) -> /LED_Data
- J4 pad 3: unconnected-(J4-Pin_3-Pad3) -> GND
- U3 pad 1: /Ext->Int/Master_CLK -> /Master_Audio_Clk
- U3 pad 26: /Exit->Int_Select -> /Int->Ext_Select
- U3 pad 5: /Ext->Int_CLK -> /Int->Ext_CLK
- U3 pad 6: /Ext->Int_In -> /Int->Ext_In
- U3 pad 7: /Ext->Int_LRC -> /Int->Ext_LRC
- U3 pad 8: /Ext->Int_Out -> /Int->Ext_Out
- U4 pad 1: /Int->Ext/Master_CLK -> /Master_Audio_Clk
- U4 pad 26: /Int->Ext_Select -> /Exit->Int_Select
- U4 pad 5: /Int->Ext_CLK -> /Ext->Int_CLK
- U4 pad 6: /Int->Ext_In -> /Ext->Int_In
- U4 pad 7: /Int->Ext_LRC -> /Ext->Int_LRC
- U4 pad 8: /Int->Ext_Out -> /Ext->Int_Out
Routing:
- net GNDA: track 0.00 -> 56.6 mm, vias 0 -> 2
- net +3V3A: track 2.25 -> 44.0 mm, vias 3 -> 5
- net Net-(U3-LOUT1): track 0.00 -> 37.2 mm, vias 0 -> 2
- net Net-(U3-LINPUT1): track 0.00 -> 26.3 mm, vias 0 -> 2
- net /Master_Audio_Clk: track 0.00 -> 25.9 mm, vias 0 -> 2
- net Net-(U3-RINPUT1): track 0.00 -> 25.8 mm, vias 0 -> 2
- net /SPI_CLK: track 0.00 -> 23.6 mm, vias 0 -> 2
- net Net-(U3-ROUT1): track 0.00 -> 23.3 mm, vias 0 -> 2
- net /MOSI: track 0.00 -> 22.7 mm, vias 0 -> 2
- net Net-(U4-LOUT1): track 2.40 -> 23.3 mm, vias 0 -> 2
- net Net-(U4-RINPUT1): track 0.00 -> 20.5 mm, vias 0 -> 2
- net GND: track 4.76 -> 25.2 mm, vias 1 -> 6
- net /Ext->Int_CLK: track 0.00 -> 20.2 mm
- net /Ext->Int_In: track 0.00 -> 19.1 mm
- net /Ext->Int_Out: track 0.00 -> 18.8 mm
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Other:
- board text added: "CosplayCore V1.0"
- board text added: "You like printed circuit boards, don't you?"

Commit message: silkscreen
Parts:
- J3: footprint Connector_JST:JST_XH_S5B-XH-A_1x05_P2.50mm_Horizontal -> Connector_JST:JST_EH_S5B-EH_1x05_P2.50mm_Horizontal
- J4: footprint Connector_JST:JST_XH_S3B-XH-A_1x03_P2.50mm_Horizontal -> Connector_JST:JST_EH_S3B-EH_1x03_P2.50mm_Horizontal
- J5: footprint Connector_JST:JST_XH_S2B-XH-A_1x02_P2.50mm_Horizontal -> Connector_JST:JST_EH_S2B-EH_1x02_P2.50mm_Horizontal
- J6: value Left_Mic -> Left_Speaker; footprint Connector_JST:JST_XH_S2B-XH-A_1x02_P2.50mm_Horizontal -> Connector_JST:JST_EH_S2B-EH_1x02_P2.50mm_Horizontal
- J7: value Right_Speaker -> Left_Speaker; footprint Connector_JST:JST_XH_S2B-XH-A_1x02_P2.50mm_Horizontal -> Connector_JST:JST_EH_S2B-EH_1x02_P2.50mm_Horizontal
- J8: value Right_Mic -> Left_Speaker; footprint Connector_JST:JST_XH_S2B-XH-A_1x02_P2.50mm_Horizontal -> Connector_JST:JST_EH_S2B-EH_1x02_P2.50mm_Horizontal
- moved J3 10.0 mm to (165.6, 96.8), turned to -90 degrees
- moved J4 5.00 mm to (130.4, 101.8), turned to 90 degrees
- moved J7 2.60 mm to (165.6, 79.1), turned to -90 degrees
- moved J6 2.50 mm to (130.4, 90.5), turned to 90 degrees
- moved J8 2.50 mm to (165.6, 88.0), turned to -90 degrees
- moved J5 2.40 mm to (130.4, 81.6), turned to 90 degrees
Connections:
- J3 pad 3: /Out_CLK -> /Out_DAT
- J3 pad 4: /Out_DAT -> /Out_CLK
Routing:
- net /Out_CLK: track 10.2 -> 13.0 mm
- net /Out_DAT: track 10.2 -> 12.7 mm
